File: Expansions/FlashBreakout/Flash.kicad_pcb (KiCad board)
At the start: 2 copper layers, 17.5 x 21.3 mm, 6 parts, among them J1 Conn_01x08_Pin, U2 W25Q128JVS

Commit message: add expansion modules
Parts:
- D1: footprint LED_SMD:LED_0402_1005Metric -> LED_SMD:LED_0603_1608Metric
- R2: value R -> 1K
- moved R1 10.1 mm to (69.6, 135.6), turned to 0 degrees
- moved C1 8.08 mm to (69.4, 128.9), turned to -45 degrees
- moved D1 1.08 mm to (69.2, 125.6)
- moved R2 0.22 mm to (70.4, 123.8), turned to 135 degrees
Routing:
- net Net-(J1-Pin_1): track 14.7 -> 3.14 mm
- net Net-(U2-~{CS}): track 4.65 -> 14.6 mm
- net GND: track 23.3 -> 19.7 mm, vias 0 -> 2
- net Net-(D1-A): track 0.98 -> 1.62 mm
Other:
- board size 17.5 x 21.3 mm -> 15.6 x 21.3 mm
