File: Expansions/FlashBreakout/Flash.kicad_sch (KiCad schematic)
At the start: 6 parts, among them J1 Conn_01x08_Pin, U2 W25Q128JVS

Commit message: add expansion modules
Parts:
- D1: footprint LED_SMD:LED_0402_1005Metric -> LED_SMD:LED_0603_1608Metric
Changed lines of the file:
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@@
 			)
 		)
-		(property "Footprint" "LED_SMD:LED_0402_1005Metric"
+		(property "Footprint" "LED_SMD:LED_0603_1608Metric"
 			(at 140.97 109.22 0)
 			(hide yes)
