File: ULTRASprig.kicad_pcb (KiCad board)
At the start: 2 copper layers, 167.6 x 51.3 mm, 36 parts, among them J1 Conn_01x10, J10 Conn_01x02, J11 Conn_01x04_Pin, J12 Conn_01x04_Pin, J13 Conn_01x07_Pin, J2 Conn_01x10, J3 Conn_01x12, J4 Conn_01x06, J5 Conn_01x08_Pin, J6 Conn_01x02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

Commit message: add expansion modules
Parts:
- added C15: 100nF, Capacitor_SMD:C_0402_1005Metric, F.Cu at (204.2, 98.8)
- added C16: 100nF, Capacitor_SMD:C_0402_1005Metric, F.Cu at (204.2, 99.8)
- added R2: 1K, Resistor_SMD:R_0603_1608Metric, B.Cu at (164.2, 71.2)
- added R3: 1M, Resistor_SMD:R_0603_1608Metric, F.Cu at (208.2, 99.5)
- added SW10: SW_Push, Button_Switch_SMD:SW_Push_1P1T_NO_CK_KMR2, B.Cu at (167.8, 72.8)
Routing:
- net Net-(R2-Pad2): track 0.00 -> 7.02 mm
- net GND: track 170.4 -> 176.6 mm, vias 1 -> 2
- net /CS: track 16.7 -> 20.1 mm

Commit message: more stuff
Parts:
- SW9: footprint Button_Switch_SMD:SW_SPST_B3S-1100 -> Button_Switch_SMD:SW_DIP_SPSTx01_Slide_Omron_A6S-110x_W8.9mm_P2.54mm
- moved SW10 26.6 mm to (192.0, 61.5), turned to 0 degrees
- moved R2 0.71 mm to (164.8, 70.8)
- moved SW9 0.25 mm to (234.3, 66.0), turned to 180 degrees
Routing:
- net Net-(R2-Pad2): track 7.02 -> 31.8 mm
- net Net-(J10-Pin_2): track 15.3 -> 4.39 mm
- net /B-: track 16.4 -> 9.86 mm, vias 1 -> 0
- net GND: track 176.6 -> 175.2 mm
- net /IO21: track 14.3 -> 13.6 mm
