File: ULTRASprig.kicad_sch (KiCad schematic)
At the start: 33 parts, among them J10 Conn_01x02, J11 Conn_01x04_Pin, J12 Conn_01x04_Pin, J13 Conn_01x07_Pin, J5 Conn_01x08_Pin, J7 Conn_01x08_Pin, J8 Conn_01x04_Pin, J9 Conn_01x04_Pin, SW1 SW_Push, SW2 SW_Push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

Commit message: add expansion modules
Parts:
- added R2: 1K, Resistor_SMD:R_0603_1608Metric, symbol Device:R
- added SW10: SW_Push, Button_Switch_SMD:SW_Push_1P1T_NO_CK_KMR2, symbol Switch:SW_Push
Connections:
- net CS: now also R2.1
- net GND: now also SW10.2
- new net: R2.2, SW10.1
Other:
- sheet CoreRP2354B renamed RPBreakout
- sheet RPBreakout: file untitled.kicad_sch -> Breakout.kicad_sch

Commit message: more stuff
Parts:
- added U1: SS12D10G5, easyeda2kicad:SW-TH_SHOU-HAN_SS12D10G4, symbol easyeda2kicad:SS12D10G5
Changed lines of the file:
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@@
+	)
+	(symbol
+		(lib_id "easyeda2kicad:SS12D10G5")
+		(at 157.48 111.76 0)
+		(unit 1)
+		(body_style 1)
+		(exclude_from_sim no)
+		(in_bom yes)
+		(on_board yes)
+		(in_pos_files yes)
+		(dnp no)
+		(fields_autoplaced yes)
+		(property "Reference" "U1"
+			(at 162.56 108.8399 0)
+			(show_name no)
+			(do_not_autoplace no)
+			(effects
+				(font
+					(size 1.27 1.27)
+				)
+				(justify left)
+			)
+		)
+		(property "Value" "SS12D10G5"
+			(at 162.56 111.3799 0)
+			(show_name no)
+			(do_not_autoplace no)
+			(effects
+				(font
+					(size 1.27 1.27)
+				)
+				(justify left)
+			)
+		)
+		(property "Footprint" "easyeda2kicad:SW-TH_SHOU-HAN_SS12D10G4"
+			(at 157.48 123.19 0)
+			(hide yes)
+			(show_name no)
+			(do_not_autoplace no)
+			(effects
+				(font
+					(size 1.27 1.27)
+				)
+			)
+		)
+		(property "Datasheet" "https://www.lcsc.com/datasheet/C7431054.pdf"
+			(at 157.48 125.73 0)
+			(hide yes)
+			(show_name no)
+			(do_not_autoplace no)
+			(effects
+				(font
+					(size 1.27 1.27)
+				)
+			)
+		)
+		(property "Description" ""
+			(at 157.48 111.76 0)
+			(hide yes)
+			(show_name no)
+			(do_not_autoplace no)
+			(effects
+				(font
+					(size 1.27 1.27)
+				)
+			)
+		)
+		(property "Manufacturer" "SHOU HAN(首韩)"
+			(at 157.48 128.27 0)
+			(hide yes)
+			(show_name no)
+			(do_not_autoplace no)
+			(effects
+				(font
+					(size 1.27 1.27)
+				)
+			)
+		)
+		(property "MPN" "SS12D10G5"
+			(at 157.48 130.81 0)
+			(hide yes)
+			(show_name no)
+			(do_not_autoplace no)
+			(effects
+				(font
+					(size 1.27 1.27)
+				)
+			)
+		)
+		(property "LCSC Part" "C7431054"
+			(at 157.48 133.35 0)
+			(hide yes)
+			(show_name no)
+			(do_not_autoplace no)
+			(effects
+				(font
+					(size 1.27 1.27)
+				)
+			)
+		)
+		(pin "2"
+		)
+		(pin "1"
+		)
+		(pin "3"
+		)
+		(instances
+			(project "ULTRASprig"
+				(path "/dc8507cf-781c-4d60-b864-1d9c098e6b00"
+					(reference "U1")
+					(unit 1)
+				)
+			)
+		)
 	)
 	(symbol
