File: core_board/RP2354B/RP2354B.kicad_sch (KiCad schematic)
At the start: 48 parts, among them J1 Conn_01x06_Pin, J10 Conn_01x10_Pin, J2 USB_C_Receptacle_USB2.0_14P, J3 Conn_01x02_Pin, J4 Conn_01x12_Pin, J6 Conn_01x10_Pin, SW2 SW_Push, U1 RP2354B, U2 USBLC6-2P6, U3 BQ24230RGT, U4 TPS62130A, Y1 Crystal_GND24

Commit message: remove extra files
Parts:
- removed C1, C2: 15pF, Capacitor_SMD:C_0402_1005Metric, symbol Device:C
- removed C10, C4, C5, C6, C8, C9: 4.7uF, Capacitor_SMD:C_0402_1005Metric, symbol Device:C
- removed C11, C12, C13, C14, C18, C19, C7: 100nF, Capacitor_SMD:C_0402_1005Metric, symbol Device:C
- removed C20, C3: 1uF, Capacitor_SMD:C_0402_1005Metric, symbol Device:C
- removed C21: 22uF, Capacitor_SMD:C_0402_1005Metric, symbol Device:C
- removed C22: 10uF, Capacitor_SMD:C_0402_1005Metric, symbol Device:C
- removed C23: 3.3nF, Capacitor_SMD:C_0402_1005Metric, symbol Device:C
- removed C24: 0.1uF, Capacitor_SMD:C_0402_1005Metric, symbol Device:C
- removed J1: Conn_01x06_Pin, Connector_PinHeader_2.54mm:PinHeader_1x06_P2.54mm_Vertical, symbol Connector:Conn_01x06_Pin
- removed J10, J6: Conn_01x10_Pin, Connector_PinHeader_2.54mm:PinHeader_1x10_P2.54mm_Vertical, symbol Connector:Conn_01x10_Pin
- removed J2: USB_C_Receptacle_USB2.0_14P, Connector_USB:USB_C_Receptacle_HRO_TYPE-C-31-M-12, symbol Connector:USB_C_Receptacle_USB2.0_14P
- removed J3: Conn_01x02_Pin, Connector_PinHeader_2.54mm:PinHeader_1x02_P2.54mm_Vertical, symbol Connector:Conn_01x02_Pin
- removed J4: Conn_01x12_Pin, Connector_PinSocket_2.54mm:PinSocket_1x12_P2.54mm_Vertical, symbol Connector:Conn_01x12_Pin
- removed L1: 3.3u, Inductor_SMD:L_0402_1005Metric, symbol Device:L
- removed L2: L, Inductor_SMD:L_0402_1005Metric, symbol Device:L
- removed R1, R2: 22, Resistor_SMD:R_0402_1005Metric, symbol Device:R
- removed R10: 3K, Resistor_SMD:R_0402_1005Metric, symbol Device:R
- removed R11: 4.4K, Resistor_SMD:R_0402_1005Metric, symbol Device:R
- removed R12: 9K, Resistor_SMD:R_0402_1005Metric, symbol Device:R
- removed R13: 2K, Resistor_SMD:R_0402_1005Metric, symbol Device:R
- removed R14: 100K, Resistor_SMD:R_0402_1005Metric, symbol Device:R
- removed R4, R8, R9: 1K, Resistor_SMD:R_0402_1005Metric, symbol Device:R
- removed R5, R7: 5.1K, Resistor_SMD:R_0402_1005Metric, symbol Device:R
- removed R6: 33, Resistor_SMD:R_0402_1005Metric, symbol Device:R
- removed SW2: SW_Push, symbol Switch:SW_Push
- removed U1: RP2354B, Package_DFN_QFN:QFN-80-1EP_10x10mm_P0.4mm_EP3.4x3.4mm, symbol MCU_RaspberryPi:RP2354B
- removed U2: USBLC6-2P6, Package_TO_SOT_SMD:SOT-666, symbol Power_Protection:USBLC6-2P6
- removed U3: BQ24230RGT, Package_DFN_QFN:VQFN-16-1EP_3x3mm_P0.5mm_EP1.68x1.68mm_ThermalVias, symbol Power_Management:BQ24230RGT
- removed U4: TPS62130A, Package_DFN_QFN:VQFN-16-1EP_3x3mm_P0.5mm_EP1.68x1.68mm_ThermalVias, symbol Regulator_Switching:TPS62130A
- removed Y1: Crystal_GND24, Crystal:Crystal_SMD_3225-4Pin_3.2x2.5mm, symbol Device:Crystal_GND24
Connections:
- no-connect marks 6 -> 0
Other:
- note removed: "Buck Converter"
- note removed: "Crystal"
- note removed: "USB-C"
- note removed: "Voltage Regulator (Internal)"

Commit message: add RP2354 BoM
Parts:
- added C1, C2: 15pF, Capacitor_SMD:C_0402_1005Metric, symbol Device:C
- added C10, C4, C5, C6, C8, C9: 4.7uF, Capacitor_SMD:C_0402_1005Metric, symbol Device:C
- added C11, C12, C13, C14, C18, C19, C7: 100nF, Capacitor_SMD:C_0402_1005Metric, symbol Device:C
- added C20, C3: 1uF, Capacitor_SMD:C_0402_1005Metric, symbol Device:C
- added C21: 22uF, Capacitor_SMD:C_0402_1005Metric, symbol Device:C
- added C22: 10uF, Capacitor_SMD:C_0402_1005Metric, symbol Device:C
- added C23: 3.3nF, Capacitor_SMD:C_0402_1005Metric, symbol Device:C
- added C24: 0.1uF, Capacitor_SMD:C_0402_1005Metric, symbol Device:C
- added J1: Conn_01x06_Pin, Connector_PinHeader_2.54mm:PinHeader_1x06_P2.54mm_Vertical, symbol Connector:Conn_01x06_Pin
- added J10, J6: Conn_01x10_Pin, Connector_PinHeader_2.54mm:PinHeader_1x10_P2.54mm_Vertical, symbol Connector:Conn_01x10_Pin
- added J2: USB_C_Receptacle_USB2.0_14P, Connector_USB:USB_C_Receptacle_HRO_TYPE-C-31-M-12, symbol Connector:USB_C_Receptacle_USB2.0_14P
- added J3: Conn_01x02_Pin, Connector_PinHeader_2.54mm:PinHeader_1x02_P2.54mm_Vertical, symbol Connector:Conn_01x02_Pin
- added J4: Conn_01x12_Pin, Connector_PinSocket_2.54mm:PinSocket_1x12_P2.54mm_Vertical, symbol Connector:Conn_01x12_Pin
- added L1: 3.3u, Inductor_SMD:L_0402_1005Metric, symbol Device:L
- added L2: L, Inductor_SMD:L_0402_1005Metric, symbol Device:L
- added R1, R2: 22, Resistor_SMD:R_0402_1005Metric, symbol Device:R
- added R10: 3K, Resistor_SMD:R_0402_1005Metric, symbol Device:R
- added R11: 4.4K, Resistor_SMD:R_0402_1005Metric, symbol Device:R
- added R12: 8K, Resistor_SMD:R_0402_1005Metric, symbol Device:R
- added R13: 25K, Resistor_SMD:R_0603_1608Metric, symbol Device:R
- added R14: 100K, Resistor_SMD:R_0402_1005Metric, symbol Device:R
- added R4, R8, R9: 1K, Resistor_SMD:R_0402_1005Metric, symbol Device:R
- added R5, R7: 5.1K, Resistor_SMD:R_0402_1005Metric, symbol Device:R
- added R6: 33, Resistor_SMD:R_0402_1005Metric, symbol Device:R
- added SW2: SW_Push, symbol Switch:SW_Push
- added U1: RP2354B, Package_DFN_QFN:QFN-80-1EP_10x10mm_P0.4mm_EP3.4x3.4mm, symbol MCU_RaspberryPi:RP2354B
- added U2: USBLC6-2P6, Package_TO_SOT_SMD:SOT-666, symbol Power_Protection:USBLC6-2P6
- added U3: BQ24230RGT, Package_DFN_QFN:VQFN-16-1EP_3x3mm_P0.5mm_EP1.68x1.68mm_ThermalVias, symbol Power_Management:BQ24230RGT
- added U4: TPS62130A, Package_DFN_QFN:VQFN-16-1EP_3x3mm_P0.5mm_EP1.68x1.68mm_ThermalVias, symbol Regulator_Switching:TPS62130A
- added Y1: Crystal_GND24, Crystal:Crystal_SMD_3225-4Pin_3.2x2.5mm, symbol Device:Crystal_GND24
Connections:
- new net: R4.1, SW2.2
- new net: C23.1, C24.2, U4.9 (SS/TR)
- new net: C5.1, J3.1 (Pin_1), U3.2 (BAT), U3.3 (BAT)
- new net: R10.2, U3.12 (ILIM)
- new net: R11.2, U3.16 (ISET)
- new net: R14.2, U4.4 (PG)
- new net: R12.1, R13.2, U4.5 (FB)
- new net: J10.1 (Pin_1), U1.12 (GPIO13)
- new net: J10.10 (Pin_10), U1.1 (GPIO4)
- new net: J10.2 (Pin_2), U1.11 (GPIO12)
- new net: J10.3 (Pin_3), U1.9 (GPIO11)
- new net: J10.4 (Pin_4), U1.8 (GPIO10)
- new net: J10.5 (Pin_5), U1.7 (GPIO9)
- new net: J10.6 (Pin_6), U1.6 (GPIO8)
- new net: J10.7 (Pin_7), U1.4 (GPIO7)
- new net: J10.8 (Pin_8), U1.3 (GPIO6)
- new net: J10.9 (Pin_9), U1.2 (GPIO5)
- new net: J2.A5 (CC1), R7.1
- new net: J2.B5 (CC2), R5.1
- new net: J4.1 (Pin_1), U1.40 (GPIO32)
- new net: J4.10 (Pin_10), U1.23 (GPIO23)
- new net: J4.11 (Pin_11), U1.22 (GPIO22)
- new net: J4.12 (Pin_12), U1.21 (GPIO21)
- new net: J4.2 (Pin_2), U1.39 (GPIO31)
- new net: J4.3 (Pin_3), U1.38 (GPIO30)
- new net: J4.4 (Pin_4), U1.37 (GPIO29)
- new net: J4.5 (Pin_5), U1.36 (GPIO28)
- new net: J4.6 (Pin_6), U1.28 (GPIO27)
- new net: J4.7 (Pin_7), U1.27 (GPIO26)
- new net: J4.8 (Pin_8), U1.26 (GPIO25)
- new net: J4.9 (Pin_9), U1.25 (GPIO24)
- new net +1V1: C10.1, C11.1, C18.1, C19.1, C20.1, C6.1, C7.1, L1.1, U1.10 (DVDD), U1.32 (DVDD), U1.51 (DVDD), U1.65 (VREG_FB)
- new net +3V3: C12.1, C13.1, C14.1, C21.1, C9.1, L2.2, R13.1, R6.1, U1.15 (IOVDD), U1.24 (IOVDD), U1.29 (IOVDD), U1.41 (IOVDD), U1.5 (IOVDD), U1.50 (IOVDD), U1.59 (ADC_AVDD), U1.60 (IOVDD), U1.64 (VREG_VIN), U1.68 (USB_OTP_VDD), U1.69 (QSPI_IOVDD), U1.76 (IOVDD)
- new net CHG: R8.1, U1.57 (GPIO46/ADC6), U3.9 (CHG)
- new net CS1: J6.5 (Pin_5), U1.49 (GPIO40/ADC0)
- new net CS2: J6.3 (Pin_3), U1.52 (GPIO41/ADC1)
- new net CS3: J6.2 (Pin_2), U1.53 (GPIO42/ADC2)
- new net CS4: J6.1 (Pin_1), U1.54 (GPIO43/ADC3)
- new net D+: R2.1, U2.4 (I/O2)
- new net D-: R1.1, U2.6 (I/O1)
- new net DN: R2.2, U1.67 (USB_DP)
- new net DP: R1.2, U1.66 (USB_DM)
- new net GND: C1.2, C10.2, C11.2, C12.2, C13.2, C14.2, C18.2, C19.2, C2.2, C20.2, C21.2, C22.2, C23.2, C3.2, C4.2, C5.2, C6.2, C7.2, C8.2, C9.2, J2.A1 (GND), J2.A12 (GND), J2.B1 (GND), J2.B12 (GND), J2.SH (SHIELD), J3.2 (Pin_2), R10.1, R11.1, R12.2, R5.2, R7.2, SW2.1, U1.62 (VREG_PGND), U1.81 (GND), U2.2 (GND), U3.1 (TS), U3.14 (TMR), U3.15 (TD), U3.4 (CE), U3.6 (EN1), U4.15 (GND), U4.16 (GND), U4.17 (GND), U4.6 (GND), U4.7 (FSW), U4.8 (DEF), Y1.2 (G), Y1.4 (G)
- new net IO1: J6.10 (Pin_10), U1.42 (GPIO33)
- new net PGD: R9.1, U1.58 (GPIO47/ADC7), U3.7 (PGOOD)
- new net RST: R4.2, U1.35 (RUN)
- new net SCLK: J1.2 (Pin_2), U1.71 (QSPI_SCLK)
- new net SD0: J1.3 (Pin_3), U1.72 (QSPI_SD0)
- new net SD1: J1.5 (Pin_5), U1.74 (QSPI_SD1)
- new net SD2: J1.4 (Pin_4), U1.73 (QSPI_SD2)
- new net SD3: J1.1 (Pin_1), U1.70 (QSPI_SD3)
- new net SPI0_MISO: J6.7 (Pin_7), U1.47 (GPIO38)
- new net SPI0_MOSI: J6.6 (Pin_6), U1.48 (GPIO39)
- new net SPI1_MISO: J6.8 (Pin_8), U1.46 (GPIO37)
- new net SPI1_MOSI: J6.9 (Pin_9), U1.45 (GPIO36)
- new net SS: J1.6 (Pin_6), U1.75 (~{QSPI_SS})
- new net USBD+: J2.A6 (D+), J2.B6 (D+), U2.3 (I/O2)
- new net USBD-: J2.A7 (D-), J2.B7 (D-), U2.1 (I/O1)
- new net VBUCK: C22.1, C24.1, C4.1, R8.2, R9.2, U3.10 (OUT), U3.11 (OUT), U3.5 (EN2), U4.10 (VIN), U4.11 (VIN), U4.12 (VIN), U4.13 (EN)
- new net VBUS: C3.1, J2.A4 (VBUS), J2.A9 (VBUS), J2.B4 (VBUS), J2.B9 (VBUS), U2.5 (VBUS), U3.13 (IN)
- new net VOUT: J6.4 (Pin_4), L2.1, R14.1, U4.1 (SW), U4.14 (VOS), U4.2 (SW), U4.3 (SW)
- new net VREGAVDD: C8.1, R6.2, U1.61 (VREG_AVDD)
- new net VREGlX: L1.2, U1.63 (VREG_LX)
- new net VSS: U3.17 (VSS), U3.8 (VSS)
- new net XIN: C1.1, U1.30 (XIN), Y1.1
- new net XOUT: C2.1, U1.31 (XOUT), Y1.3
- no-connect marks 0 -> 6
Other:
- note added: "Buck Converter"
- note added: "Crystal"
- note added: "USB-C"
- note added: "Voltage Regulator (Internal)"
