File: Mainboard/ULTRASprig.kicad_pcb (KiCad board)
At the start: 2 copper layers, 167.6 x 51.3 mm, 41 parts, among them J1 Conn_01x10, J10 Conn_01x02, J11 Conn_01x04_Pin, J12 Conn_01x04_Pin, J13 Conn_01x07_Pin, J2 Conn_01x10, J3 Conn_01x12, J4 Conn_01x06, J5 Conn_01x08_Pin, J6 Conn_01x02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

Commit message: update stupid nbs
Parts:
- added J14: Conn_01x02, Connector_PinHeader_2.54mm:PinHeader_1x02_P2.54mm_Vertical, F.Cu at (200.0, 104.3)
- SW9: footprint Button_Switch_SMD:SW_DIP_SPSTx01_Slide_Omron_A6S-110x_W8.9mm_P2.54mm -> Button_Switch_SMD:SW_SPST_B3S-1100
Routing:
- net Net-(J14-Pin_2): track 0.00 -> 7.72 mm
- net Net-(J14-Pin_1): track 0.00 -> 5.27 mm
- net GND: track 175.2 -> 174.2 mm
